File: kicad/PortaRe0/usb_hub.kicad_sch (KiCad schematic)
At the start: 0 parts

Commit message: session07: VL812 usb_hubシート完成・power回路修正
- VL812 usb_hubシート完成
  - 電源ピン・デカップリングC配置
  - USB3.0 TX側ACカップリング・USB2.0直結
  - SPI Flash（W25Q32）接続・プルダウン
  - 水晶発振子（25MHz）追加
  - USBHOC1#/2# プルアップ追加（過電流誤検知防止）
- power回路: SCL/SDA/USB_DP/USB_DM GlobalLabel追加
- VL812データシート追加

Co-Authored-By: Claude Sonnet 4.6 <noreply@anthropic.com>
Parts:
- added C14, C15, C17, C20, C22, C23, C24, C25, C26, C28, C30, C32, C34, C36, C38, C41, C42, C44, C46, C47, C52, C53, C58, C59, C66, C67: 100nF, symbol Device:C_Small
- added C16, C18, C19, C21: 10μF, symbol Device:C_Small
- added C27, C29, C31, C33, C35, C37, C39, C40, C43, C45: 10pF, symbol Device:C_Small
- added C48: 4.7μF, symbol Device:C_Small
- added L3: 4.7μH, symbol Device:L_Small
- added R12, R16, R17, R19, R25: 10KΩ, symbol Device:R_Small
- added R13, R14, R15, R20, R21, R22, R23, R24: 100KΩ, symbol Device:R_Small
- added R18: 200Ω, symbol Device:R_Small
- added U4: VL812, PortaRe0:QFN-76_L9.0-W9.0-P0.40-BL-EP, symbol PortaRe0:VL812
- added U5: W25Q32JVSSIQ, PortaRe0:SOIC-8_L5.3-W5.3-P1.27-LS8.0-BL, symbol PortaRe0:W25Q32JVSSIQ
- added Y1: 25MHz, symbol Device:Crystal_Small
Connections:
- new net: C58.2, U4.66 (SSTX2+)
- new net: R15.2, U4.53 (USBHGRN1)
- new net: R17.2, U5.7 (IO3)
- new net: R24.2, U4.50 (USBHGRN4)
- new net: R19.2, U4.54 (~{RESET})
- new net: L3.2, U4.39 (LX)
- new net: R25.2, U4.44 (~{USBHOC2})
- new net: R12.2, U4.45 (~{USBHOC1})
- new net: R16.2, U5.3 (IO2)
- new net: R22.2, U4.52 (USBHGRN2)
- new net: C46.1, U4.22 (SSTX0-)
- new net: C53.2, U4.60 (SSTX1-)
- new net: R23.2, U4.51 (USBHGRN3)
- new net: C59.2, U4.67 (SSTX2-)
- new net: C47.1, U4.23 (SSTX0+)
- new net: R18.2, U4.1 (SSREXT)
- new net: C52.2, U4.59 (SSTX1+)
- new net 1V2_HUB: C15.2, C16.2, C17.2, C18.2, C19.2, C20.2, C21.2, C22.2, C32.2, C33.2, C34.2, C35.2, C36.2, C37.2, C40.2, C41.2, C42.2, C43.2, C44.2, C45.2, L3.1, U4.13 (VCCA12SSRX4), U4.24 (VCCA12SSRX0), U4.30 (VDD), U4.37 (DC12FB), U4.48 (VDD), U4.5 (VCCA12SSRX3), U4.58 (VDD), U4.61 (VCCA12SSRX1), U4.68 (VCCA12SSRX2), U4.74 (VCCA12SSM)
- new net 3V3_HUB: C14.2, C23.2, C24.2, C25.2, C26.2, C27.2, C28.2, C29.2, C30.2, C31.2, C38.2, C39.2, C48.2, C66.2, C67.2, R12.1, R16.1, R17.1, R19.1, R25.1, U4.18 (DC33FB), U4.2 (VCCA33SSM), U4.27 (VCCA33SS0), U4.36 (VSUS33), U4.41 (VSUS33), U4.49 (VSUS33), U4.71 (VCCA33SS12), U4.8 (VCCA33SS34), U5.8 (VCC)
- new net 5V_SYS: U4.19 (VCC5I), U4.31 (VBUSDET), U4.38 (VCC5I), U4.47 (EXTPWRON)
- new net GNDPWR: C14.1, C15.1, C16.1, C17.1, C18.1, C19.1, C20.1, C21.1, C22.1, C23.1, C24.1, C25.1, C26.1, C27.1, C28.1, C29.1, C30.1, C31.1, C32.1, C33.1, C34.1, C35.1, C36.1, C37.1, C38.1, C39.1, C40.1, C41.1, C42.1, C43.1, C44.1, C45.1, C48.1, C66.1, C67.1, R13.1, R14.1, R15.1, R18.1, R20.1, R21.1, R22.1, R23.1, R24.1, U4.20 (VCC12I), U4.75 (SSXI), U4.76 (SSXO), U5.4 (GND), Y1.1, Y1.2
- new net SPICS: R20.2, U4.32 (USBHMBR4), U5.1 (~{CS})
- new net SPISCLK: R13.2, U4.33 (USBHMBR3), U5.6 (CLK)
- new net SPISI: R14.2, U4.34 (USBHMBR2), U5.5 (DI（IO0）)
- new net SPISO: R21.2, U4.35 (USBHMBR1), U5.2 (DO（IO1）)
- new net USB2_DP1_DM: U4.65 (USBHP1-)
- new net USB2_DP1_DP: U4.64 (USBHP1+)
- new net USB2_DP2_DM: U4.73 (USBHP2-)
- new net USB2_DP2_DP: U4.72 (USBHP2+)
- new net USB2_RP_DM: U4.10 (USBHP3-)
- new net USB2_RP_DP: U4.9 (USBHP3+)
- new net USB2_UP_DM: U4.29 (USBDP-)
- new net USB2_UP_DP: U4.28 (USBDP+)
- new net USB3_DP1_RX_N: U4.63 (SSRX1-)
- new net USB3_DP1_RX_P: U4.62 (SSRX1+)
- new net USB3_DP1_TX_N: C53.1
- new net USB3_DP1_TX_P: C52.1
- new net USB3_DP2_RX_N: U4.70 (SSRX2-)
- new net USB3_DP2_RX_P: U4.69 (SSRX2+)
- new net USB3_DP2_TX_N: C59.1
- new net USB3_DP2_TX_P: C58.1
- new net USB3_UP_RX_N: U4.25 (SSRX0-)
- new net USB3_UP_RX_P: U4.26 (SSRX0+)
- new net USB3_UP_TX_N: C46.2
- new net USB3_UP_TX_P: C47.2
