File: kicad/PortaRe0/connectors.kicad_sch (KiCad schematic)
At the start: 0 parts

Commit message: KiCad: connectorsシート更新（J_HDMI_CTRL・J_SBC_USB1・J_SBC_USB2配置・配線）
Co-Authored-By: Claude Sonnet 4.6 <noreply@anthropic.com>
Parts:
- added FPC1: J_HDMI_CTRL, PortaRe0:FPC-SMD_24P-P0.50_FPC-05F-24PH20, symbol PortaRe0:FPC-05F-24PH20
- added R52, R53: 5.1KΩ, symbol Device:R_Small
- added R54, R55: 22KΩ, symbol Device:R_Small
- added USBC2: J_SBC_USB1, PortaRe0:USB-C-SMD_TYPE-C-USB-3, symbol PortaRe0:TYPE-C3.1_C168690
- added USBC3: J_SBC_USB2, PortaRe0:USB-C-SMD_TYPE-C-USB-3, symbol PortaRe0:TYPE-C3.1_C168690
Connections:
- new net: R55.2, USBC3.B5
- new net: R53.2, USBC2.A5
- new net: R54.2, USBC3.A5
- new net: R52.2, USBC2.B5
- new net 5V_SYS: FPC1.18, FPC1.22, FPC1.23, FPC1.24, R54.1, R55.1, USBC3.A4, USBC3.A9, USBC3.B4, USBC3.B9
- new net GNDPWR: FPC1.11, FPC1.14, FPC1.17, FPC1.2, FPC1.20, FPC1.21, FPC1.25, FPC1.26, FPC1.5, FPC1.8, R52.1, R53.1, USBC2.0, USBC2.A1, USBC2.A12, USBC2.B1, USBC2.B12, USBC3.0, USBC3.A1, USBC3.A12, USBC3.B1, USBC3.B12
- new net HDMI_CLKN: FPC1.13
- new net HDMI_CLKP: FPC1.12
- new net HDMI_D0N: FPC1.10
- new net HDMI_D0P: FPC1.9
- new net HDMI_D1N: FPC1.7
- new net HDMI_D1P: FPC1.6
- new net HDMI_D2N: FPC1.4
- new net HDMI_D2P: FPC1.3
- new net HDMI_HPD: FPC1.1, FPC1.19
- new net HDMI_SCL: FPC1.15
- new net HDMI_SDA: FPC1.16
- new net USB2_UP_DM: USBC2.A7, USBC2.B7
- new net USB2_UP_DP: USBC2.A6, USBC2.B6
- new net USB2_UP_VBUS: USBC2.A4, USBC2.A9, USBC2.B4, USBC2.B9
- new net USB3_UP_RX_N: USBC2.A3, USBC2.B3
- new net USB3_UP_RX_P: USBC2.A2, USBC2.B2
- new net USB3_UP_TX_N: USBC2.A10, USBC2.B10
- new net USB3_UP_TX_P: USBC2.A11, USBC2.B11
- no-connect marks 0 -> 16
