File: kicad/PortaRe0/keyboard.kicad_sch (KiCad schematic)
At the start: 158 parts, among them J1 StickSocket, U6 RP2040#1, Y4 C70565

Commit message: Docs: session32終了処理・ドキュメント構成整理・session_close.py作成
Parts:
- removed J1: StickSocket, PortaRe0:FPC-SMD_5034800400, symbol Connector:Conn_01x04_Socket
- removed K_SW1, K_SW2: KeyBoard, PortaRe0:KEY-SMD_4P-SKSCLXX010, symbol Switch:SW_Push
- removed K_SW10, K_SW11, K_SW12, K_SW13, K_SW14, K_SW15, K_SW16, K_SW17, K_SW18, K_SW19, K_SW20, K_SW21, K_SW22, K_SW23, K_SW24, K_SW25, K_SW26, K_SW27, K_SW28, K_SW29, K_SW3, K_SW30, K_SW31, K_SW32, K_SW33, K_SW34, K_SW35, K_SW36, K_SW37, K_SW38, K_SW39, K_SW4, K_SW40, K_SW41, K_SW42, K_SW43, K_SW44, K_SW45, K_SW46, K_SW47, K_SW48, K_SW49, K_SW5, K_SW50, K_SW51, K_SW52, K_SW53, K_SW54, K_SW55, K_SW56, K_SW57, K_SW58, K_SW59, K_SW6, K_SW60, K_SW61, K_SW62, K_SW63, K_SW7, K_SW8, K_SW9: KeyBoard, PortaRe0:KEY-SMD_4P-L4.2-W3.2-P2.20-LS4.6, symbol Switch:SW_Push
- removed K_SW64: BOOTSEL_SW, PortaRe0:KEY-SMD_4P-L4.2-W3.2-P2.20-LS4.6, symbol Switch:SW_Push
- added B_SW1: BOOTSEL_SW, PortaRe0:KEY-SMD_4P-L4.2-W3.2-P2.20-LS4.6, symbol PortaRe0:SKRPABE010
- added K_SW1, K_SW2: KeyBoard, PortaRe0:KEY-SMD_4P-SKSCLXX010, symbol PortaRe0:SKSCLBE010
- added K_SW10, K_SW11, K_SW12, K_SW13, K_SW14, K_SW15, K_SW16, K_SW17, K_SW18, K_SW19, K_SW20, K_SW21, K_SW22, K_SW23, K_SW24, K_SW25, K_SW26, K_SW27, K_SW28, K_SW29, K_SW3, K_SW30, K_SW31, K_SW32, K_SW33, K_SW34, K_SW35, K_SW36, K_SW37, K_SW38, K_SW39, K_SW4, K_SW40, K_SW41, K_SW42, K_SW43, K_SW44, K_SW45, K_SW46, K_SW47, K_SW48, K_SW49, K_SW5, K_SW50, K_SW51, K_SW52, K_SW53, K_SW54, K_SW55, K_SW56, K_SW57, K_SW58, K_SW59, K_SW6, K_SW60, K_SW61, K_SW62, K_SW63, K_SW64, K_SW7, K_SW8, K_SW9: KeyBoard, PortaRe0:KEY-SMD_4P-L4.2-W3.2-P2.20-LS4.6, symbol PortaRe0:SKRPABE010
- added SW_D64: 1N4148W, PortaRe0:SOD-123_L2.8-W1.8-LS3.7-RD, symbol Device:D_Small
- added Stick1: 5034800440, PortaRe0:FPC-SMD_5034800400, symbol PortaRe0:5034800440
Connections:
- net +3V3: now also Stick1.3
- net COL0: now also K_SW1.3, K_SW12.1, K_SW21.1, K_SW3.1, K_SW30.1, K_SW39.1, K_SW48.1, K_SW57.1
- net COL1: now also K_SW13.1, K_SW22.1, K_SW31.1, K_SW4.1, K_SW40.1, K_SW49.1, K_SW58.1
- net COL2: now also K_SW14.1, K_SW23.1, K_SW32.1, K_SW41.1, K_SW5.1, K_SW50.1, K_SW59.1
- net COL3: now also K_SW15.1, K_SW24.1, K_SW33.1, K_SW42.1, K_SW51.1, K_SW6.1, K_SW60.1
- net COL4: now also K_SW16.1, K_SW25.1, K_SW34.1, K_SW43.1, K_SW52.1, K_SW61.1, K_SW7.1
- net COL5: now also K_SW17.1, K_SW26.1, K_SW35.1, K_SW44.1, K_SW53.1, K_SW62.1, K_SW8.1
- net COL6: now also K_SW18.1, K_SW27.1, K_SW36.1, K_SW45.1, K_SW54.1, K_SW63.1, K_SW9.1
- net COL7: now also K_SW10.1, K_SW19.1, K_SW28.1, K_SW37.1, K_SW46.1, K_SW55.1, K_SW64.1
- net COL8: now also K_SW11.1, K_SW2.3, K_SW20.1, K_SW29.1, K_SW38.1, K_SW47.1, K_SW56.1
- net GND: now also B_SW1.4, Stick1.1, Stick1.5, Stick1.6
- net QSPI_SS: now also B_SW1.2
- net ROW7: now also SW_D64.1 (K)
- net STICK_X: now also Stick1.2
- net STICK_Y: now also Stick1.4
- net at SW_D39.2 (A): now also K_SW39.3
- net at SW_D7.2 (A): now also K_SW7.3
- net at SW_D58.2 (A): now also K_SW58.3
- net at SW_D12.2 (A): now also K_SW12.3
- net at SW_D22.2 (A): now also K_SW22.3
- net at SW_D19.2 (A): now also K_SW19.3
- net at SW_D15.2 (A): now also K_SW15.3
- net at SW_D4.2 (A): now also K_SW4.3
- net at SW_D17.2 (A): now also K_SW17.3
- net at SW_D47.2 (A): now also K_SW47.3
- net at SW_D20.2 (A): now also K_SW20.3
- net at SW_D9.2 (A): now also K_SW9.3
- net at SW_D24.2 (A): now also K_SW24.3
- net at SW_D38.2 (A): now also K_SW38.3
- net at SW_D21.2 (A): now also K_SW21.3
- net at SW_D1.2 (A): now also K_SW1.1
- net at SW_D42.2 (A): now also K_SW42.3
- net at SW_D8.2 (A): now also K_SW8.3
- net at SW_D45.2 (A): now also K_SW45.3
- net at SW_D41.2 (A): now also K_SW41.3
- net at SW_D48.2 (A): now also K_SW48.3
- net at SW_D35.2 (A): now also K_SW35.3
- net at SW_D49.2 (A): now also K_SW49.3
- net at SW_D54.2 (A): now also K_SW54.3
- net at SW_D14.2 (A): now also K_SW14.3
- net at SW_D37.2 (A): now also K_SW37.3
- net at SW_D18.2 (A): now also K_SW18.3
- net at SW_D53.2 (A): now also K_SW53.3
- net at SW_D25.2 (A): now also K_SW25.3
- net at SW_D23.2 (A): now also K_SW23.3
- net at SW_D52.2 (A): now also K_SW52.3
- net at SW_D44.2 (A): now also K_SW44.3
- net at SW_D28.2 (A): now also K_SW28.3
- net at SW_D31.2 (A): now also K_SW31.3
- net at SW_D10.2 (A): now also K_SW10.3
- net at SW_D50.2 (A): now also K_SW50.3
- net at SW_D34.2 (A): now also K_SW34.3
- net at SW_D33.2 (A): now also K_SW33.3
- net at SW_D61.2 (A): now also K_SW61.3
- net at SW_D56.2 (A): now also K_SW56.3
- net at SW_D36.2 (A): now also K_SW36.3
- net at SW_D51.2 (A): now also K_SW51.3
- net at SW_D40.2 (A): now also K_SW40.3
- net at SW_D29.2 (A): now also K_SW29.3
- net at SW_D30.2 (A): now also K_SW30.3
- net at SW_D16.2 (A): now also K_SW16.3
- net at SW_D62.2 (A): now also K_SW62.3
- net at SW_D57.2 (A): now also K_SW57.3
- net at SW_D43.2 (A): now also K_SW43.3
- net at SW_D55.2 (A): now also K_SW55.3
- net at SW_D59.2 (A): now also K_SW59.3
- net at SW_D3.2 (A): now also K_SW3.3
- net at SW_D11.2 (A): now also K_SW11.3
- net at SW_D27.2 (A): now also K_SW27.3
- net at SW_D26.2 (A): now also K_SW26.3
- net at SW_D6.2 (A): now also K_SW6.3
- net at SW_D60.2 (A): now also K_SW60.3
- net at SW_D46.2 (A): now also K_SW46.3
- net at SW_D63.2 (A): now also K_SW63.3
- net at SW_D2.2 (A): now also K_SW2.1
- net at SW_D13.2 (A): now also K_SW13.3
- net at SW_D32.2 (A): now also K_SW32.3
- net at SW_D5.2 (A): now also K_SW5.3
- new net: K_SW64.3, SW_D64.2 (A)
- no-connect marks 3 -> 133
Other:
- moved on the sheet: D2, D3, D4, R31, R32, R33, SW_D1, SW_D10, SW_D11, SW_D12, SW_D13, SW_D14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

Commit message: Docs: session34終了処理・0402化確定・ディスプレイ調査・PCBレイアウト進行中
Parts:
- C49, C50, C51, C54, C55, C56, C57, C60, C61, C62, C63, C64, C65, C68, C69: footprint Capacitor_SMD:C_0603_1608Metric -> Capacitor_SMD:C_0402_1005Metric
- R26, R29, R30, R31, R32, R33, R34: footprint Resistor_SMD:R_0603_1608Metric -> Resistor_SMD:R_0402_1005Metric
Changed lines of the file:
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@@
 			)
 		)
-		(property "Footprint" "Capacitor_SMD:C_0603_1608Metric"
+		(property "Footprint" "Capacitor_SMD:C_0402_1005Metric"
 			(at 62.23 173.99 0)
 			(effects
@@
 			)
 		)
-		(property "Footprint" "Capacitor_SMD:C_0603_1608Metric"
+		(property "Footprint" "Capacitor_SMD:C_0402_1005Metric"
 			(at 99.06 105.41 0)
 			(effects
@@
 			)
 		)
-		(property "Footprint" "Capacitor_SMD:C_0603_1608Metric"
+		(property "Footprint" "Capacitor_SMD:C_0402_1005Metric"
 			(at 104.14 105.41 0)
 			(effects
@@
 			)
 		)
-		(property "Footprint" "Capacitor_SMD:C_0603_1608Metric"
+		(property "Footprint" "Capacitor_SMD:C_0402_1005Metric"
 			(at 90.17 83.82 0)
 			(effects
@@
 			)
 		)
-		(property "Footprint" "Capacitor_SMD:C_0603_1608Metric"
+		(property "Footprint" "Capacitor_SMD:C_0402_1005Metric"
 			(at 106.68 105.41 0)
 			(effects
@@
 			)
 		)
-		(property "Footprint" "Capacitor_SMD:C_0603_1608Metric"
+		(property "Footprint" "Capacitor_SMD:C_0402_1005Metric"
 			(at 120.65 105.41 0)
 			(effects
@@
 			)
 		)
-		(property "Footprint" "Resistor_SMD:R_0603_1608Metric"
+		(property "Footprint" "Resistor_SMD:R_0402_1005Metric"
 			(at 124.46 114.3 0)
 			(effects
@@
 			)
 		)
-		(property "Footprint" "Capacitor_SMD:C_0603_1608Metric"
+		(property "Footprint" "Capacitor_SMD:C_0402_1005Metric"
 			(at 109.22 105.41 0)
 			(effects
@@
 			)
 		)
-		(property "Footprint" "Capacitor_SMD:C_0603_1608Metric"
+		(property "Footprint" "Capacitor_SMD:C_0402_1005Metric"
 			(at 114.3 105.41 0)
 			(effects
@@
 			)
 		)
-		(property "Footprint" "Capacitor_SMD:C_0603_1608Metric"
+		(property "Footprint" "Capacitor_SMD:C_0402_1005Metric"
 			(at 116.84 105.41 0)
 			(effects
@@
 			)
 		)
-		(property "Footprint" "Resistor_SMD:R_0603_1608Metric"
+		(property "Footprint" "Resistor_SMD:R_0402_1005Metric"
 			(at 72.39 260.35 0)
 			(effects
@@
 			)
 		)
-		(property "Footprint" "Capacitor_SMD:C_0603_1608Metric"
+		(property "Footprint" "Capacitor_SMD:C_0402_1005Metric"
 			(at 95.25 105.41 0)
 			(effects
@@
 			)
 		)
-		(property "Footprint" "Capacitor_SMD:C_0603_1608Metric"
+		(property "Footprint" "Capacitor_SMD:C_0402_1005Metric"
 			(at 62.23 179.07 0)
 			(effects
@@
 			)
 		)
-		(property "Footprint" "Resistor_SMD:R_0603_1608Metric"
+		(property "Footprint" "Resistor_SMD:R_0402_1005Metric"
 			(at 68.58 191.77 0)
 			(effects
@@
 			)
 		)
-		(property "Footprint" "Capacitor_SMD:C_0603_1608Metric"
+		(property "Footprint" "Capacitor_SMD:C_0402_1005Metric"
 			(at 87.63 105.41 0)
 			(effects
@@
 			)
 		)
-		(property "Footprint" "Resistor_SMD:R_0603_1608Metric"
+		(property "Footprint" "Resistor_SMD:R_0402_1005Metric"
 			(at 72.39 254 0)
 			(effects
@@
 			)
 		)
-		(property "Footprint" "Capacitor_SMD:C_0603_1608Metric"
+		(property "Footprint" "Capacitor_SMD:C_0402_1005Metric"
 			(at 90.17 105.41 0)
 			(effects
@@
 			)
 		)
-		(property "Footprint" "Capacitor_SMD:C_0603_1608Metric"
+		(property "Footprint" "Capacitor_SMD:C_0402_1005Metric"
 			(at 128.27 114.3 0)
 			(effects
@@
 			)
 		)
-		(property "Footprint" "Resistor_SMD:R_0603_1608Metric"
+		(property "Footprint" "Resistor_SMD:R_0402_1005Metric"
 			(at 127 86.36 0)
 			(effects
@@
 			)
 		)
-		(property "Footprint" "Resistor_SMD:R_0603_1608Metric"
+		(property "Footprint" "Resistor_SMD:R_0402_1005Metric"
 			(at 72.39 139.7 0)
 			(effects
@@
 			)
 		)
-		(property "Footprint" "Resistor_SMD:R_0603_1608Metric"
+		(property "Footprint" "Resistor_SMD:R_0402_1005Metric"
 			(at 72.39 266.7 0)
 			(effects
@@
 			)
 		)
-		(property "Footprint" "Capacitor_SMD:C_0603_1608Metric"
+		(property "Footprint" "Capacitor_SMD:C_0402_1005Metric"
 			(at 111.76 105.41 0)
 			(effects
