File: kicad/PortaRe0/power.kicad_sch (KiCad schematic)
At the start: 44 parts, among them J4 Battery, SW1 SW_START, SW2 KillSW, U1 BQ25895RTWR, U2 TPS61023DRLR, U3 AP2112K-3.3TRG1

Commit message: Docs: session32終了処理・ドキュメント構成整理・session_close.py作成
Parts:
- removed SW1: SW_START, PortaRe0:KEY-SMD_4P-SKSCLXX010, symbol Switch:SW_SPST
- added SW1: SW_START, PortaRe0:KEY-SMD_4P-SKSCLXX010, symbol PortaRe0:SKSCLBE010
Connections:
- net VSYS: now also SW1.3
- net at D8.1 (A), R14.1: now also SW1.1
- no-connect marks 7 -> 9
Changed lines of the file:
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@@
 		(at 300.99 45.72)
 	)
+	(no_connect
+		(at 261.62 43.18)
+	)
+	(no_connect
+		(at 266.7 43.18)
+	)
 	(wire
 		(pts
@@
 	(wire
 		(pts
-			(xy 256.54 58.42) (xy 259.08 58.42)
+			(xy 256.54 58.42) (xy 261.62 58.42)
 		)
 		(stroke
@@
 	(wire
 		(pts
+			(xy 266.7 58.42) (xy 281.94 58.42)
+		)
+		(stroke
+			(width 0)
+			(type default)
+		)
+	)
+	(wire
+		(pts
 			(xy 152.4 69.85) (xy 152.4 71.12)
 		)
@@
 	(wire
 		(pts
-			(xy 269.24 58.42) (xy 281.94 58.42)
-		)
-		(stroke
-			(width 0)
-			(type default)
-		)
-	)
-	(wire
-		(pts
 			(xy 134.62 76.2) (xy 143.51 76.2)
 		)
@@
 	)
 	(symbol
+		(lib_id "PortaRe0:SKSCLBE010")
+		(at 262.89 50.8 90)
+		(unit 1)
+		(exclude_from_sim no)
+		(in_bom yes)
+		(on_board yes)
+		(dnp no)
+		(property "Reference" "SW1"
+			(at 268.478 47.244 0)
+			(effects
+				(font
+					(size 1.27 1.27)
+				)
+				(justify right)
+			)
+		)
+		(property "Value" "SW_START"
+			(at 260.096 46.482 0)
+			(effects
+				(font
+					(size 1.27 1.27)
+				)
+				(justify right)
+			)
+		)
+		(property "Footprint" "PortaRe0:KEY-SMD_4P-SKSCLXX010"
+			(at 274.32 50.8 0)
+			(effects
+				(font
+					(size 1.27 1.27)
+				)
+				(hide yes)
+			)
+		)
+		(property "Datasheet" "https://lcsc.com/product-detail/Tactile-Switches_ALPS_SKSCLBE010_3-3-5-1-1-Side-press-1-6N_C115361.html"
+			(at 276.86 50.8 0)
+			(effects
+				(font
+					(size 1.27 1.27)
+				)
+				(hide yes)
+			)
+		)
+		(property "Description" ""
+			(at 262.89 50.8 0)
+			(effects
+				(font
+					(size 1.27 1.27)
+				)
+				(hide yes)
+			)
+		)
+		(property "LCSC Part" "C115361"
+			(at 279.4 50.8 0)
+			(effects
+				(font
+					(size 1.27 1.27)
+				)
+				(hide yes)
+			)
+		)
+		(pin "3"
+		)
+		(pin "2"
+		)
+		(pin "4"
+		)
+		(pin "1"
+		)
+		(instances
+			(project "PortaRe0"
+				(path "/479aadc4-f9a0-4ec2-b000-6a17237038f1/bbdd0b45-407f-430f-96c4-71b6262b4665"
+					(reference "SW1")
+					(unit 1)
+				)
+			)
+		)
+	)
+	(symbol
 		(lib_id "power:GNDPWR")
 		(at 313.69 88.9 0)
@@
 					(unit 1)
 				)
-			)
-		)
-	)
-	(symbol
-		(lib_id "Switch:SW_SPST")
-		(at 264.16 58.42 0)
-		(unit 1)
-		(exclude_from_sim no)
-		(in_bom yes)
-		(on_board yes)
-		(dnp no)
-		(property "Reference" "SW1"
-			(at 264.16 54.102 0)
-			(effects
-				(font
-					(size 1.27 1.27)
-				)
-			)
-		)
-		(property "Value" "SW_START"
-			(at 264.16 55.626 0)
-			(effects
-				(font
-					(size 1.27 1.27)
-				)
-			)
-		)
-		(property "Footprint" "PortaRe0:KEY-SMD_4P-SKSCLXX010"
-			(at 264.16 58.42 0)
-			(effects
-				(font
-					(size 1.27 1.27)
-				)
-				(hide yes)
-			)
-		)
-		(property "Datasheet" "~"
-			(at 264.16 58.42 0)
-			(effects
-				(font
-					(size 1.27 1.27)
-				)
-				(hide yes)
-			)
-		)
-		(property "Description" "Single Pole Single Throw (SPST) switch"
-			(at 264.16 58.42 0)
-			(effects
-				(font
-					(size 1.27 1.27)
-				)
-				(hide yes)
-			)
-		)
-		(pin "1"
-		)
-		(pin "2"
-		)
-		(instances
-			(project "PortaRe0"
-				(path "/479aadc4-f9a0-4ec2-b000-6a17237038f1/bbdd0b45-407f-430f-96c4-71b6262b4665"
-					(reference "SW1")
-					(unit 1)
-				)

Commit message: Docs: session34終了処理・0402化確定・ディスプレイ調査・PCBレイアウト進行中
Parts:
- removed J4: Battery, PortaRe0:CONN-TH_S8B-PH-K-S-LF-SN, symbol Connector:Conn_01x08_Socket
- added J1: Battery, PortaRe0:CONN_BM06B-ACHFKS-GACN-ETF_JST, symbol PortaRe0:BM06B-ACHFKS-GACN-ETFLFSN
- C11, C114, C12, C2, C4, C5, C7, C9: footprint Capacitor_SMD:C_0603_1608Metric -> Capacitor_SMD:C_0402_1005Metric
- R1, R10, R11, R14, R2, R21, R3, R4, R48, R49, R6, R64, R7: footprint Resistor_SMD:R_0603_1608Metric -> Resistor_SMD:R_0402_1005Metric
Connections:
- net +BATT: now also J1.1, J1.2, J1.3
- net GND: now also J1.4, J1.5, J1.6
