File: kicad/PortaRe0/PortaRe0.kicad_pcb (KiCad board)
At the start: 6 copper layers, 135 x 77 mm, 357 parts, among them J1 Battery, J9 PJ-307C, Q1 BSS138, SW1 SW_START, SW2 KillSW, U1 BQ25895RTWR, U10 TPS2042BDR, U11 RP2040#2, U12 HC-USB3.0-L168-WP, U13 PCM5102APWR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

Commit message: Docs: Session41終了処理・PROGRESS/index/README更新・ガーバー・CPL追加
Parts:
- moved SW_D2 1.04 mm to (188.4, 49.1)
- moved K_SW2 0.74 mm to (188.4, 45.2)
- moved K_SW1 0.58 mm to (64.5, 45.2)
- moved SW_D1 0.58 mm to (64.5, 49.1)
Routing:
- net /keyboard/COL8: track 178.9 -> 220.0 mm
- net /keyboard/COL0: track 268.6 -> 286.7 mm, vias 7 -> 8
- net /keyboard/ROW0: track 171.7 -> 169.9 mm, vias 4 -> 3
- net Net-(SW_D2-A): track 6.89 -> 5.37 mm
Other:
- outline, holes or cut-outs redrawn
